File: board.sch (EAGLE design)
At the start: 6 parts

Commit message: v1.1
Parts:
- U$1, U$2: value TERMINAL10 -> KF141V-2.54-10P; device terminals:TERMINAL10 -> terminals:KF141V-2.54-10P
Connections:
- net GND: now also U$1.P$1
Changed lines of the file:
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@@
 </variantdefs>
 <classes>
-<class number="0" name="default" width="1.27" drill="0">
+<class number="0" name="default" width="1.27" drill="0.381">
 <clearance class="0" value="0.381"/>
 </class>
-<class number="1" name="VCC" width="1.778" drill="0">
+<class number="1" name="VCC" width="1.778" drill="0.381">
 <clearance class="0" value="0.381"/>
 </class>
@@
 <parts>
 <part name="PRO_MICRO" library="SparkFun-Boards" deviceset="SPARKFUN_PRO_MICRO" device="" value="PRO_MICRO"/>
-<part name="U$1" library="terminals" deviceset="TERMINAL10" device=""/>
-<part name="U$2" library="terminals" deviceset="TERMINAL10" device=""/>
+<part name="U$1" library="terminals" deviceset="KF141V-2.54-10P" device=""/>
+<part name="U$2" library="terminals" deviceset="KF141V-2.54-10P" device=""/>
 <part name="U$3" library="terminals" deviceset="TERMINAL4" device=""/>
 <part name="R1" library="rcl" library_urn="urn:adsk.eagle:library:334" deviceset="R-EU_" device="0207/10" package3d_urn="urn:adsk.eagle:package:23491/2" value="10K"/>
@@
 <part name="SUPPLY2" library="supply2" library_urn="urn:adsk.eagle:library:372" deviceset="GND" device=""/>
 <part name="SUPPLY3" library="supply2" library_urn="urn:adsk.eagle:library:372" deviceset="GND" device=""/>
+<part name="SUPPLY4" library="supply2" library_urn="urn:adsk.eagle:library:372" deviceset="GND" device=""/>
 </parts>
 <sheets>
@@
 <attribute name="VALUE" x="50.8" y="35.56" size="1.778" layer="96"/>
 </instance>
-<instance part="U$1" gate="G$1" x="-25.4" y="66.04" smashed="yes" rot="R180"/>
-<instance part="U$2" gate="G$1" x="144.78" y="60.96" smashed="yes"/>
+<instance part="U$1" gate="G$1" x="-25.4" y="63.5" smashed="yes" rot="R180"/>
+<instance part="U$2" gate="G$1" x="144.78" y="63.5" smashed="yes"/>
 <instance part="U$3" gate="G$1" x="43.18" y="20.32" smashed="yes" rot="R270"/>
 <instance part="R1" gate="G$1" x="63.5" y="78.74" smashed="yes">
@@
 <instance part="SUPPLY3" gate="GND" x="40.64" y="68.58" smashed="yes" rot="R180">
 <attribute name="VALUE" x="42.545" y="71.755" size="1.778" layer="96" rot="R180"/>
+</instance>
+<instance part="SUPPLY4" gate="GND" x="5.08" y="38.1" smashed="yes">
+<attribute name="VALUE" x="3.175" y="34.925" size="1.778" layer="96"/>
 </instance>
 </instances>
@@
 <wire x1="30.48" y1="58.42" x2="30.48" y2="86.36" width="0.1524" layer="91"/>
 <pinref part="U$1" gate="G$1" pin="P$10"/>
-<wire x1="30.48" y1="86.36" x2="5.08" y2="86.36" width="0.1524" layer="91"/>
+<wire x1="30.48" y1="86.36" x2="-22.86" y2="86.36" width="0.1524" layer="91"/>
 </segment>
 </net>
@@
 <wire x1="27.94" y1="55.88" x2="27.94" y2="81.28" width="0.1524" layer="91"/>
 <pinref part="U$1" gate="G$1" pin="P$9"/>
-<wire x1="27.94" y1="81.28" x2="5.08" y2="81.28" width="0.1524" layer="91"/>
+<wire x1="27.94" y1="81.28" x2="-22.86" y2="81.28" width="0.1524" layer="91"/>
 </segment>
 </net>
@@
 <wire x1="25.4" y1="53.34" x2="25.4" y2="76.2" width="0.1524" layer="91"/>
 <pinref part="U$1" gate="G$1" pin="P$8"/>
-<wire x1="25.4" y1="76.2" x2="5.08" y2="76.2" width="0.1524" layer="91"/>
+<wire x1="25.4" y1="76.2" x2="-22.86" y2="76.2" width="0.1524" layer="91"/>
 </segment>
 </net>
@@
 <wire x1="22.86" y1="50.8" x2="22.86" y2="71.12" width="0.1524" layer="91"/>
 <pinref part="U$1" gate="G$1" pin="P$7"/>
-<wire x1="22.86" y1="71.12" x2="5.08" y2="71.12" width="0.1524" layer="91"/>
+<wire x1="22.86" y1="71.12" x2="-22.86" y2="71.12" width="0.1524" layer="91"/>
 </segment>
 </net>
@@
 <wire x1="20.32" y1="48.26" x2="20.32" y2="66.04" width="0.1524" layer="91"/>
 <pinref part="U$1" gate="G$1" pin="P$6"/>
-<wire x1="20.32" y1="66.04" x2="5.08" y2="66.04" width="0.1524" layer="91"/>
+<wire x1="20.32" y1="66.04" x2="-22.86" y2="66.04" width="0.1524" layer="91"/>
 </segment>
 </net>
@@
 <wire x1="48.26" y1="45.72" x2="17.78" y2="45.72" width="0.1524" layer="91"/>
 <wire x1="17.78" y1="45.72" x2="17.78" y2="60.96" width="0.1524" layer="91"/>
-<wire x1="17.78" y1="60.96" x2="5.08" y2="60.96" width="0.1524" layer="91"/>
+<wire x1="17.78" y1="60.96" x2="-22.86" y2="60.96" width="0.1524" layer="91"/>
 </segment>
 </net>
@@
 <pinref part="U$1" gate="G$1" pin="P$4"/>
 <wire x1="15.24" y1="43.18" x2="15.24" y2="55.88" width="0.1524" layer="91"/>
-<wire x1="15.24" y1="55.88" x2="5.08" y2="55.88" width="0.1524" layer="91"/>
+<wire x1="15.24" y1="55.88" x2="-22.86" y2="55.88" width="0.1524" layer="91"/>
 </segment>
 </net>
@@
 <pinref part="U$1" gate="G$1" pin="P$3"/>
 <wire x1="12.7" y1="40.64" x2="12.7" y2="50.8" width="0.1524" layer="91"/>
-<wire x1="12.7" y1="50.8" x2="5.08" y2="50.8" width="0.1524" layer="91"/>
+<wire x1="12.7" y1="50.8" x2="-22.86" y2="50.8" width="0.1524" layer="91"/>
 </segment>
 </net>
@@
 <pinref part="PRO_MICRO" gate="G$1" pin="*10"/>
 <pinref part="U$2" gate="G$1" pin="P$10"/>
-<wire x1="71.12" y1="40.64" x2="114.3" y2="40.64" width="0.1524" layer="91"/>
+<wire x1="71.12" y1="40.64" x2="142.24" y2="40.64" width="0.1524" layer="91"/>
 </segment>
 </net>
@@
 <pinref part="U$2" gate="G$1" pin="P$9"/>
 <wire x1="86.36" y1="50.8" x2="86.36" y2="45.72" width="0.1524" layer="91"/>
-<wire x1="86.36" y1="45.72" x2="114.3" y2="45.72" width="0.1524" layer="91"/>
+<wire x1="86.36" y1="45.72" x2="142.24" y2="45.72" width="0.1524" layer="91"/>
 </segment>
 </net>
@@
 <wire x1="91.44" y1="53.34" x2="91.44" y2="50.8" width="0.1524" layer="91"/>
 <pinref part="U$2" gate="G$1" pin="P$8"/>
-<wire x1="91.44" y1="50.8" x2="114.3" y2="50.8" width="0.1524" layer="91"/>
+<wire x1="91.44" y1="50.8" x2="142.24" y2="50.8" width="0.1524" layer="91"/>
 </segment>
 </net>
@@
 <segment>
 <pinref part="PRO_MICRO" gate="G$1" pin="A2"/>
-<wire x1="71.12" y1="55.88" x2="114.3" y2="55.88" width="0.1524" layer="91"/>
+<wire x1="71.12" y1="55.88" x2="142.24" y2="55.88" width="0.1524" layer="91"/>
 <pinref part="U$2" gate="G$1" pin="P$7"/>
 </segment>
@@
 <pinref part="U$2" gate="G$1" pin="P$6"/>
 <wire x1="96.52" y1="58.42" x2="96.52" y2="60.96" width="0.1524" layer="91"/>
-<wire x1="96.52" y1="60.96" x2="114.3" y2="60.96" width="0.1524" layer="91"/>
+<wire x1="96.52" y1="60.96" x2="142.24" y2="60.96" width="0.1524" layer="91"/>
 </segment>
 </net>
@@
 <wire x1="81.28" y1="60.96" x2="91.44" y2="60.96" width="0.1524" layer="91"/>
 <wire x1="91.44" y1="60.96" x2="91.44" y2="66.04" width="0.1524" layer="91"/>
-<wire x1="91.44" y1="66.04" x2="114.3" y2="66.04" width="0.1524" layer="91"/>
+<wire x1="91.44" y1="66.04" x2="142.24" y2="66.04" width="0.1524" layer="91"/>
 <wire x1="71.12" y1="60.96" x2="81.28" y2="60.96" width="0.1524" layer="91"/>
 <junction x="81.28" y="60.96"/>
@@
 <pinref part="U$2" gate="G$1" pin="P$1"/>
 <pinref part="U$2" gate="G$1" pin="P$2"/>
-<wire x1="114.3" y1="81.28" x2="114.3" y2="86.36" width="0.1524" layer="91"/>
-<junction x="114.3" y="81.28"/>
-<wire x1="114.3" y1="76.2" x2="114.3" y2="81.28" width="0.1524" layer="91"/>
+<wire x1="142.24" y1="81.28" x2="142.24" y2="86.36" width="0.1524" layer="91"/>
+<junction x="142.24" y="81.28"/>
+<wire x1="142.24" y1="76.2" x2="142.24" y2="81.28" width="0.1524" layer="91"/>
 <pinref part="U$2" gate="G$1" pin="P$3"/>
-<junction x="114.3" y="76.2"/>
-<wire x1="114.3" y1="71.12" x2="114.3" y2="76.2" width="0.1524" layer="91"/>
+<junction x="142.24" y="76.2"/>
+<wire x1="142.24" y1="71.12" x2="142.24" y2="76.2" width="0.1524" layer="91"/>
 <pinref part="U$2" gate="G$1" pin="P$4"/>
-<wire x1="114.3" y1="71.12" x2="99.06" y2="71.12" width="0.1524" layer="91"/>
+<wire x1="142.24" y1="71.12" x2="99.06" y2="71.12" width="0.1524" layer="91"/>
 <wire x1="99.06" y1="71.12" x2="86.36" y2="71.12" width="0.1524" layer="91"/>
 <wire x1="86.36" y1="71.12" x2="86.36" y2="66.04" width="0.1524" layer="91"/>
-<junction x="114.3" y="71.12"/>
+<junction x="142.24" y="71.12"/>
 <pinref part="PRO_MICRO" gate="G$1" pin="GND@2"/>
 <wire x1="86.36" y1="66.04" x2="78.74" y2="66.04" width="0.1524" layer="91"/>
-<junction x="114.3" y="86.36"/>
+<junction x="142.24" y="86.36"/>
 <pinref part="SUPPLY2" gate="GND" pin="GND"/>
 <junction x="99.06" y="71.12"/>
@@
 <junction x="40.64" y="63.5"/>
 </segment>
-</net>
+<segment>
+<pinref part="U$1" gate="G$1" pin="P$1"/>
+<pinref part="SUPPLY4" gate="GND" pin="GND"/>
+<wire x1="5.08" y1="40.64" x2="-22.86" y2="40.64" width="0.1524" layer="91"/>
+</segment>
+</net>
